File: kicad/usbwledc.kicad_sch (KiCad schematic)
At the start: 26 parts, among them J1 5V PAD, J10 USB_C_Receptacle_USB2.0, J2 D1 PAD, J3 GND PAD, J4 5V PAD, J5 D2 PAD, J6 GND PAD, J7 Accessories, SW1 FLASH_SW, U1 CH340N, U2 AMS1117-3.3, U3 ESP32-WROOM-32

Commit message: update to Revision 1.2
Updated:
ESP32-WROOM-32 to ESP32-WROOM-32E
Changed CH340N to CH340C with Auto reset function
Changed components from 0805 to 0603/0402
Updated JLCPC component C8 to C7469983

Added:
SN74LVC2T45DCUR Levelshifter from 3.3V to 5V
USB Data ESD protection
Parts:
- removed U1: CH340N, Package_SO:SOP-8_3.9x4.9mm_P1.27mm, symbol Interface_USB:CH340X
- added C10, C9: 100nF, Capacitor_SMD:C_0402_1005Metric, symbol Device:C
- added D1: SP0503BAHT, Package_TO_SOT_SMD:SOT-143, symbol Power_Protection:SP0503BAHT
- added J8, J9: Conn_01x03_Pin, Connector_PinHeader_2.54mm:PinHeader_1x03_P2.54mm_Vertical, symbol Connector:Conn_01x03_Pin
- added Q1, Q2: L8050QLT1G, Package_TO_SOT_SMD:SOT-23, symbol Transistor_BJT:SS8050
- added R6, R7: 10k, Resistor_SMD:R_0402_1005Metric, symbol Device:R
- added U4: SN74LVC2T45DCUR, Package_SO:VSSOP-8_2.3x2mm_P0.5mm, symbol Logic_LevelTranslator:SN74LVC2T45DCUR
- added U5: CH340C, Package_SO:SOIC-16_3.9x9.9mm_P1.27mm, symbol Interface_USB:CH340C
- C1, C2, C4: footprint Capacitor_SMD:C_0603_1608Metric -> Capacitor_SMD:C_0402_1005Metric; LCSC (none) -> C1525; MPN C14663 -> C1525
- C3, C5, C7: footprint Capacitor_SMD:C_0805_2012Metric -> Capacitor_SMD:C_0603_1608Metric; LCSC (none) -> C96446; MPN C15850 -> C96446
- C6: footprint Capacitor_SMD:C_0603_1608Metric -> Capacitor_SMD:C_0402_1005Metric; LCSC (none) -> C52923; MPN C15849 -> C52923
- C8: LCSC (none) -> C7469983; MPN C131115 -> C7469983
- J10: LCSC (none) -> C2988369
- MK1: LCSC (none) -> C5142171
- R1: footprint Resistor_SMD:R_0603_1608Metric -> Resistor_SMD:R_0402_1005Metric; LCSC (none) -> C25741; MPN C25803 -> C25741
- R2, R3: footprint Resistor_SMD:R_0603_1608Metric -> Resistor_SMD:R_0402_1005Metric; LCSC (none) -> C1525; MPN C25804 -> C1525
- R4, R5: LCSC (none) -> C23186
- SW1: LCSC (none) -> C318884
- U2: LCSC (none) -> C6186
- U3: value ESP32-WROOM-32 -> ESP32-WROOM-32E-N4; footprint RF_Module:ESP32-WROOM-32 -> RF_Module:ESP32-WROOM-32E; Aliexpress https://de.aliexpress.com/item/32840441199.html -> (none); LCSC (none) -> C701341; Mouser 356-ESP32WRM32E132PH -> (none)
Connections:
- net +3V3: now also R2.2, C10.1, U4.8 (VCCB), U5.16 (VCC), U5.4 (V3); no longer R2.1
- net +5V: now also C9.1, J8.1 (Pin_1), J9.1 (Pin_1), U4.1 (VCCA)
- net D+: now also D1.2 (K), U5.5 (UD+)
- net D-: now also D1.3 (K), U5.6 (UD-)
- net FLASH: now also R2.1, Q2.2 (E); no longer R2.2
- net GND: now also C10.2, C9.2, D1.1 (A), J8.3 (Pin_3), J9.3 (Pin_3), U4.4 (GND), U4.5 (DIR), U5.1 (GND)
- net RX: now also U5.2 (TXD)
- net STRIP_DATA_1: now also U4.7 (B1); no longer J2.1 (Pin_1)
- net STRIP_DATA_2: now also U4.6 (B2); no longer J5.1 (Pin_1)
- net TX: now also U5.3 (RXD)
- net EN: now reaches C6.1, R3.2, U3.3 (EN)
- net EN: now also Q1.3 (C)
- new net: Q2.1 (B), R7.2
- new net: Q1.1 (B), R6.2
- new net DTR: Q2.3 (C), R6.1, U5.13 (~{DTR})
- new net RTS: Q1.2 (E), R7.1, U5.14 (~{RTS})
- new net STRIP_DATA_LS_1: J2.1 (Pin_1), J8.2 (Pin_2), U4.2 (A1)
- new net STRIP_DATA_LS_2: J5.1 (Pin_1), J9.2 (Pin_2), U4.3 (A2)
- no-connect marks 24 -> 29
Other:
- company: NANDXOR -> Yannik25
- moved on the sheet: C2, C4, C5, C6, U3

Commit message: fix resistor placement instead of caps, replace mic, fix count of components
Parts:
- removed MK1: GSA4737, microphone:Microphone-6pin, symbol microphone:GSA4737
- added MK1: ICS-43434, Sensor_Audio:InvenSense_ICS-43434-6_3.5x2.65mm, symbol Sensor_Audio:ICS-43434
- R2, R3, R6, R7: LCSC C1525 -> C25531; MPN C1525 -> C25531
Connections:
- net +3V3: now also MK1.5 (VDD)
- net DTR: now also Q2.2 (E); no longer Q2.3 (C)
- net FLASH: now also Q2.3 (C); no longer Q2.2 (E)
- net GND: now also MK1.2 (LR), MK1.3 (GND)
- net I2S_SCK: now also MK1.4 (SCK)
- net I2S_SD: now also MK1.6 (SD)
